File: PSK_kicad/Pincher_Split_Keyboard.kicad_pcb (KiCad board)
At the start: 2 copper layers, 114.9 x 60.9 mm, 20 parts, among them U1 RP2040_Zero, U2 TRRS

Commit message: fixed rx tx
Parts:
- added U3: TRRS, Footprints:Jack_3.5mm_PJ320D_Horizontal, B.Cu at (197.4, 96.6)
- U2: footprint Footprints:TRRS_PJ-320A -> Footprints:Jack_3.5mm_PJ320D_Horizontal
- moved U2 3.43 mm to (197.4, 96.6), turned to -135 degrees
- moved S17 1.52 mm to (180.0, 94.8)
- moved S16 1.25 mm to (144.0, 89.8)
- moved S18 0.76 mm to (162.0, 92.3)
Connections:
- U1 pad 3: SW11 -> SW10
- U1 pad 4: SW10 -> SW11
- U1 pad 7: SW14 -> TMB2
- U1 pad 8: TMB2 -> TMB3
- U1 pad 9: TMB3 -> SW14
Routing:
- net SW10: track 80.0 -> 93.2 mm
- net SW14: track 125.7 -> 115.4 mm
- net GND: track 416.8 -> 425.8 mm, vias 0 -> 1
- net SW11: track 65.1 -> 71.4 mm
- net TMB3: track 55.1 -> 61.1 mm
- net VCC: track 55.3 -> 60.2 mm, vias 0 -> 1
- net RX: track 44.1 -> 48.8 mm, vias 0 -> 1
- net TMB2: track 43.5 -> 47.0 mm
- net TX: track 51.9 -> 49.0 mm, vias 0 -> 1
- net SW15: track 113.2 -> 111.0 mm
- net SW16: track 95.6 -> 97.5 mm
