File: FrontPlate/FrontPlate.kicad_sch (KiCad schematic)
At the start: 15 parts

Commit message: better front plate
Parts:
- S1, S2, S3, S4: footprint keyswitches:PLATE_choc_footprint -> Footprints:PLATE_choc_footprint_exp
- S10, S11, S12, S13, S14, S15, S5, S6, S7, S8, S9: footprint keyswitches:PLATE_choc_footprint -> Footprints:PLATE_choc
Changed lines of the file:
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@@
 			)
 		)
-		(property "Footprint" "keyswitches:PLATE_choc_footprint"
+		(property "Footprint" "Footprints:PLATE_choc"
 			(at 48.26 83.82 0)
 			(effects
@@
 			)
 		)
-		(property "Footprint" "keyswitches:PLATE_choc_footprint"
+		(property "Footprint" "Footprints:PLATE_choc_footprint_exp"
 			(at 96.52 69.85 0)
 			(effects
@@
 			)
 		)
-		(property "Footprint" "keyswitches:PLATE_choc_footprint"
+		(property "Footprint" "Footprints:PLATE_choc"
 			(at 81.28 83.82 0)
 			(effects
@@
 			)
 		)
-		(property "Footprint" "keyswitches:PLATE_choc_footprint"
+		(property "Footprint" "Footprints:PLATE_choc"
 			(at 48.26 97.79 0)
 			(effects
@@
 			)
 		)
-		(property "Footprint" "keyswitches:PLATE_choc_footprint"
+		(property "Footprint" "Footprints:PLATE_choc"
 			(at 97.79 83.82 0)
 			(effects
@@
 			)
 		)
-		(property "Footprint" "keyswitches:PLATE_choc_footprint"
+		(property "Footprint" "Footprints:PLATE_choc"
 			(at 114.3 69.85 0)
 			(effects
@@
 			)
 		)
-		(property "Footprint" "keyswitches:PLATE_choc_footprint"
+		(property "Footprint" "Footprints:PLATE_choc"
 			(at 63.5 97.79 0)
 			(effects
@@
 			)
 		)
-		(property "Footprint" "keyswitches:PLATE_choc_footprint"
+		(property "Footprint" "Footprints:PLATE_choc"
 			(at 113.03 97.79 0)
 			(effects
@@
 			)
 		)
-		(property "Footprint" "keyswitches:PLATE_choc_footprint"
+		(property "Footprint" "Footprints:PLATE_choc"
 			(at 96.52 97.79 0)
 			(effects
@@
 			)
 		)
-		(property "Footprint" "keyswitches:PLATE_choc_footprint"
+		(property "Footprint" "Footprints:PLATE_choc_footprint_exp"
 			(at 63.5 69.85 0)
 			(effects
@@
 			)
 		)
-		(property "Footprint" "keyswitches:PLATE_choc_footprint"
+		(property "Footprint" "Footprints:PLATE_choc"
 			(at 80.01 97.79 0)
 			(effects
@@
 			)
 		)
-		(property "Footprint" "keyswitches:PLATE_choc_footprint"
+		(property "Footprint" "Footprints:PLATE_choc_footprint_exp"
 			(at 48.26 69.85 0)
 			(effects
@@
 			)
 		)
-		(property "Footprint" "keyswitches:PLATE_choc_footprint"
+		(property "Footprint" "Footprints:PLATE_choc_footprint_exp"
 			(at 80.01 69.85 0)
 			(effects
@@
 			)
 		)
-		(property "Footprint" "keyswitches:PLATE_choc_footprint"
+		(property "Footprint" "Footprints:PLATE_choc"
 			(at 64.77 83.82 0)
 			(effects
@@
 			)
 		)
-		(property "Footprint" "keyswitches:PLATE_choc_footprint"
+		(property "Footprint" "Footprints:PLATE_choc"
 			(at 116.84 83.82 0)
 			(effects
